File: STM32 GPS Tracker.kicad_pcb (KiCad board)
At the start: 4 copper layers, 43.5 x 58.5 mm, 57 parts, among them J1 Screw_Terminal_01x02, J2 LEFT HEADER PINS, J3 693010020611, J4 RIGHT HEADER PINS, Q1 AO3407A, SW1 SW_Push, SW2 SW_Push, U1 SIM808, U2 TPS5430DDA, U3 SMF05CT1G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

Commit message: Completed the Layer 1
Routing:
- added copper zone on In2.Cu, net +3.3V
- added copper zone on B.Cu, net GND
- added copper zone on F.Cu, net GND
- added copper zone on In1.Cu, net GND
Changed lines of the file:
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@@
 		)
 		(embedded_fonts no)
-		(model "AO3407A.stp"
+		(model "${KIPRJMOD}/Libraries/3D Models/SOT-23-3L_AOS.step"
 			(offset
 				(xyz 0 0 0)
@@
 			)
 			(rotate
-				(xyz 0 0 0)
+				(xyz -0 -0 90)
 			)
 		)
@@
 		)
 		(embedded_fonts no)
+		(model "${KIPRJMOD}/Libraries/3D Models/TPS5430DDA.step"
+			(offset
+				(xyz 0 0 0)
+			)
+			(scale
+				(xyz 1 1 1)
+			)
+			(rotate
+				(xyz -90 -0 -0)
+			)
+		)
 	)
 	(footprint "Resistor_SMD:R_0805_2012Metric"
@@
 		(tags "fuse")
 		(property "Reference" "F1"
-			(at -1.885 0 90)
+			(at -1.735 0.025 180)
 			(layer "F.SilkS")
 			(effects
@@
 		(tags "terminal block bornier2")
 		(property "Reference" "J1"
-			(at 2.54 -5.08 0)
+			(at -3.745 1.65 0)
 			(layer "F.SilkS")
 			(effects
@@
 		)
 		(embedded_fonts no)
-		(model "${KICAD9_3DMODEL_DIR}/TerminalBlock.3dshapes/TerminalBlock_bornier-2_P5.08mm.step"
+		(model "${KICAD9_3DMODEL_DIR}/TerminalBlock_Phoenix.3dshapes/TerminalBlock_Phoenix_MKDS-1,5-2-5.08_1x02_P5.08mm_Horizontal.step"
 			(offset
-				(xyz 2.539999962 0 0)
+				(xyz 0.04 0 0)
 			)
 			(scale
-				(xyz 1 1 1)
+				(xyz 1 0.9 0.9)
 			)
 			(rotate
-				(xyz 0 0 0)
+				(xyz -0 -0 -0)
 			)
 		)
@@
 		)
 		(embedded_fonts no)
-		(model "${KICAD9_3DMODEL_DIR}/Inductor_SMD.3dshapes/L_10.4x10.4_H4.8.step"
+		(model "${KIPRJMOD}/Libraries/3D Models/B82464P4153M000.stp"
 			(offset
 				(xyz 0 0 0)
@@
 			)
 			(rotate
-				(xyz 0 0 0)
+				(xyz 90 180 90)
 			)
 		)
@@
 	)
 	(zone
+		(net 1)
+		(net_name "GND")
+		(layers "F.Cu" "B.Cu")
+		(hatch edge 0.5)
+		(priority 2)
+		(connect_pads
+			(clearance 0.5)
+		)
+		(min_thickness 0.25)
+		(filled_areas_thickness no)
+		(fill yes
+			(thermal_gap 0.5)
+			(thermal_bridge_width 0.5)
+		)
+		(polygon
+			(pts
+				(xy 79.75 62.25) (xy 127.95 62.25) (xy 128 125.525) (xy 79.5 125.7)
+			)
+		)
+	)
+	(zone
 		(net 29)
 		(net_name "Net-(J3-CLK)")
@@
 			)
 		)
+	)
+	(zone
+		(net 1)
+		(net_name "GND")
+		(layer "In1.Cu")
+		(hatch edge 0.5)
+		(connect_pads
+			(clearance 0.5)
+		)
+		(min_thickness 0.25)
+		(filled_areas_thickness no)
+		(fill yes
+			(thermal_gap 0.5)
+			(thermal_bridge_width 0.5)
+		)
+		(polygon
+			(pts
+				(xy 80 62.5) (xy 127.5 62.5) (xy 127.5 125) (xy 80 125)
+			)
+		)
+	)
+	(zone
+		(net 2)
+		(net_name "+3.3V")
+		(layer "In2.Cu")
+		(hatch edge 0.5)
+		(priority 1)
+		(connect_pads
+			(clearance 0.5)
+		)
+		(min_thickness 0.25)
+		(filled_areas_thickness no)
+		(fill yes
+			(thermal_gap 0.5)
+			(thermal_bridge_width 0.5)
+		)
+		(polygon
+			(pts
+				(xy 80 62.5) (xy 127.5 62.5) (xy 127.5 125) (xy 80 125)
+			)
+		)
